File: jlc-katzen.kicad_sch (KiCad schematic)
At the start: 62 parts, among them J1 USB_C_Receptacle_USB2.0_16P, J2 Conn_01x04, J3 Conn_01x04, J4 Conn_01x02, J5 Conn_ARM_SWD_TagConnect_TC2030, Q1 2N7002, Q2 2N7002, Q3 2N7002, U1 XC6206P332MR, U2 W25Q128JVSIQ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

Commit message: fix sch metadata
Other:
- note removed: "FIGURE OUT HOW MANY FIT ON THE BOARD"
- title: (none) -> JLCPCB Katzenohren assembly practice board
Changed lines of the file:
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@@
 	(generator_version "8.0")
 	(paper "A3")
+	(title_block
+		(title "JLCPCB Katzenohren assembly practice board")
+		(date "2024-03-16")
+		(rev "A")
+	)
 	(junction
 		(at 50.8 27.94)
@@
 		(effects
 			(font
-				(size 1.27 1.27)
-			)
-		)
-	)
-	(text "FIGURE OUT HOW MANY FIT ON THE BOARD"
-		(exclude_from_sim no)
-		(at 322.58 59.944 0)
-		(effects
-			(font
